File: pcb/ILSS_PCB_2026_DEMO/ILSS_PCB_2026_DEMO.kicad_sch (KiCad schematic)
At the start: 115 parts, among them IC1 4691, IC10 4691, IC11 DRV2605LDGSR, IC2 4691, IC3 4691, IC4 4691, IC5 4691, IC6 4691, IC7 4691, IC8 4691, IC9 4691, J1 ERM MOTOR, J2 REAR PROG PINS, J3 SPARE GPIO, J4 UJ20-C-H-G-SMT-1-P16-TR, P1 S2B-PH-SM4-TB, Q1 DMN2058U, U1 XIAO-ESP32-S3-SMD, U2 ATECC608A-MAHDA, U3 MAX17048G_T10

Commit message: feat: schematic finalised, pcb routed
Parts:
- removed IC1, IC10, IC2, IC3, IC4, IC5, IC6, IC7, IC8, IC9: 4691, ILSS:ADAFRUIT_SK6812_SIDE_4691, symbol ILSS_LANYARD:4691
- removed LED1, LED2: IN-S63BTG, ILSS:LEDC1608X55N, symbol ILSS_LANYARD:IN-S63BTG
- removed LS1: CMT-7525-03-SMT-TR, ILSS:CMT752503SMTTR, symbol ILSS_LANYARD:CMT-7525-03-SMT-TR
- removed S1, S3: TS11-674-50-BK-160-RA-D, ILSS:SW_TS11-674-50-BK-160-RA-D, symbol ILSS_LANYARD:TS11-674-50-BK-160-RA-D
- removed S2: TS11-674-50-BK-160-RA-D, ILSS_LANYARD:SW_TS11-674-50-BK-160-RA-D, symbol ILSS_LANYARD:TS11-674-50-BK-160-RA-D
- added IC1, IC10, IC2, IC3, IC4, IC5, IC6, IC7, IC8, IC9: 4691, ILSS:ADAFRUIT_SK6812_SIDE_4691, symbol ILSS:4691
- added LED1, LED2: IN-S63BTG, ILSS:LEDC1608X55N, symbol ILSS:IN-S63BTG
- added LS1: CMT-7525-03-SMT-TR, ILSS:CMT752503SMTTR, symbol ILSS:CMT-7525-03-SMT-TR
- added S1, S2, S3: TS11-674-50-BK-160-RA-D, ILSS:SW_TS11-674-50-BK-160-RA-D, symbol ILSS:TS11-674-50-BK-160-RA-D
- J1: renamed from J3; footprint (none) -> Connector_PinHeader_2.54mm:PinHeader_1x02_P2.54mm_Vertical; now not fitted
- J2: footprint (none) -> Connector_PinHeader_2.54mm:PinHeader_1x06_P2.54mm_Vertical; now not fitted
- JP1: renamed from JP3; footprint (none) -> Jumper:SolderJumper-2_P1.3mm_Open_Pad1.0x1.5mm; symbol Jumper:SolderJumper_2_Bridged -> Jumper:SolderJumper_2_Open
- JP10: renamed from JP14; footprint (none) -> Jumper:SolderJumper-2_P1.3mm_Open_Pad1.0x1.5mm; symbol Jumper:SolderJumper_2_Bridged -> Jumper:SolderJumper_2_Open
- JP11: renamed from JP15; footprint (none) -> Jumper:SolderJumper-2_P1.3mm_Open_Pad1.0x1.5mm; symbol Jumper:SolderJumper_2_Bridged -> Jumper:SolderJumper_2_Open
- JP12: renamed from JP16; footprint (none) -> Jumper:SolderJumper-2_P1.3mm_Open_Pad1.0x1.5mm
- JP13: renamed from JP17; footprint (none) -> Jumper:SolderJumper-2_P1.3mm_Open_Pad1.0x1.5mm
- JP14: renamed from JP18; footprint (none) -> Jumper:SolderJumper-2_P1.3mm_Open_Pad1.0x1.5mm
- JP15: renamed from JP5; footprint (none) -> Jumper:SolderJumper-2_P1.3mm_Open_Pad1.0x1.5mm; symbol Jumper:SolderJumper_2_Bridged -> Jumper:SolderJumper_2_Open
- JP16: renamed from JP19; footprint (none) -> Jumper:SolderJumper-2_P1.3mm_Open_Pad1.0x1.5mm; symbol Jumper:SolderJumper_2_Bridged -> Jumper:SolderJumper_2_Open
- JP17: renamed from JP20; footprint (none) -> Jumper:SolderJumper-2_P1.3mm_Open_Pad1.0x1.5mm; symbol Jumper:SolderJumper_2_Bridged -> Jumper:SolderJumper_2_Open
- JP18: renamed from JP21; footprint (none) -> Jumper:SolderJumper-2_P1.3mm_Open_Pad1.0x1.5mm
- JP19: renamed from JP22; footprint (none) -> Jumper:SolderJumper-2_P1.3mm_Open_Pad1.0x1.5mm; symbol Jumper:SolderJumper_2_Bridged -> Jumper:SolderJumper_2_Open
- JP2: renamed from JP4; footprint (none) -> Jumper:SolderJumper-2_P1.3mm_Open_Pad1.0x1.5mm; symbol Jumper:SolderJumper_2_Bridged -> Jumper:SolderJumper_2_Open
- JP20: renamed from JP23; footprint (none) -> Jumper:SolderJumper-2_P1.3mm_Open_Pad1.0x1.5mm; symbol Jumper:SolderJumper_2_Bridged -> Jumper:SolderJumper_2_Open
- JP21: renamed from JP24; footprint (none) -> Jumper:SolderJumper-2_P1.3mm_Open_Pad1.0x1.5mm
- JP22: renamed from JP6; footprint (none) -> Jumper:SolderJumper-2_P1.3mm_Open_Pad1.0x1.5mm; symbol Jumper:SolderJumper_2_Bridged -> Jumper:SolderJumper_2_Open
- JP23: renamed from JP25; footprint (none) -> Jumper:SolderJumper-2_P1.3mm_Open_Pad1.0x1.5mm
- JP24: renamed from JP26; footprint (none) -> Jumper:SolderJumper-2_P1.3mm_Open_Pad1.0x1.5mm
- JP25: renamed from JP7; footprint (none) -> Jumper:SolderJumper-2_P1.3mm_Open_Pad1.0x1.5mm; symbol Jumper:SolderJumper_2_Bridged -> Jumper:SolderJumper_2_Open
- JP26: renamed from JP8; footprint (none) -> Jumper:SolderJumper-2_P1.3mm_Open_Pad1.0x1.5mm; symbol Jumper:SolderJumper_2_Bridged -> Jumper:SolderJumper_2_Open
- JP27: footprint (none) -> Jumper:SolderJumper-2_P1.3mm_Open_Pad1.0x1.5mm
- JP3: renamed from JP1; footprint (none) -> Jumper:SolderJumper-2_P1.3mm_Open_Pad1.0x1.5mm
- JP5: renamed from JP9; footprint (none) -> Jumper:SolderJumper-2_P1.3mm_Open_Pad1.0x1.5mm; symbol Jumper:SolderJumper_2_Bridged -> Jumper:SolderJumper_2_Open
- JP6: renamed from JP10; footprint (none) -> Jumper:SolderJumper-2_P1.3mm_Open_Pad1.0x1.5mm; symbol Jumper:SolderJumper_2_Bridged -> Jumper:SolderJumper_2_Open
- JP7: renamed from JP11; footprint (none) -> Jumper:SolderJumper-2_P1.3mm_Open_Pad1.0x1.5mm
- JP8: renamed from JP12; footprint (none) -> Jumper:SolderJumper-2_P1.3mm_Open_Pad1.0x1.5mm; symbol Jumper:SolderJumper_2_Bridged -> Jumper:SolderJumper_2_Open
- JP9: renamed from JP13; footprint (none) -> Jumper:SolderJumper-2_P1.3mm_Open_Pad1.0x1.5mm; symbol Jumper:SolderJumper_2_Bridged -> Jumper:SolderJumper_2_Open
- TP1: value RGB_LED_DIN -> RGB_LED_DIN_TP; footprint (none) -> TestPoint:TestPoint_Pad_D2.0mm
- TP10: renamed from TP13; footprint (none) -> TestPoint:TestPoint_Pad_D2.0mm
- TP11: renamed from TP14; footprint (none) -> TestPoint:TestPoint_Pad_D2.0mm
- TP12: renamed from TP15; footprint (none) -> TestPoint:TestPoint_Pad_D2.0mm
- TP13: renamed from TP3; footprint (none) -> TestPoint:TestPoint_Pad_D2.0mm
- TP14: renamed from TP16; footprint (none) -> TestPoint:TestPoint_Pad_D2.0mm
- TP15: renamed from TP4; footprint (none) -> TestPoint:TestPoint_Pad_D2.0mm
- TP16: renamed from TP5; footprint (none) -> TestPoint:TestPoint_Pad_D2.0mm
- TP2: footprint (none) -> TestPoint:TestPoint_Pad_D2.0mm
- TP3: renamed from TP6; footprint (none) -> TestPoint:TestPoint_Pad_D2.0mm
- TP4: renamed from TP7; footprint (none) -> TestPoint:TestPoint_Pad_D2.0mm
- TP5: renamed from TP8; footprint (none) -> TestPoint:TestPoint_Pad_D2.0mm
- TP6: renamed from TP9; footprint (none) -> TestPoint:TestPoint_Pad_D2.0mm
- TP7: renamed from TP10; footprint (none) -> TestPoint:TestPoint_Pad_D2.0mm
- TP8: renamed from TP11; footprint (none) -> TestPoint:TestPoint_Pad_D2.0mm
- TP9: renamed from TP12; footprint (none) -> TestPoint:TestPoint_Pad_D2.0mm
- renumbered C3 to C1, C1 to C2, C2 to C3, D2 to D1, D1 to D2, J4 to J3, J1 to J4, JP2 to JP4, R4 to R1, R9 to R10, R10 to R11, R11 to R12, R12 to R13, R13 to R14, R14 to R15, R15 to R16, R5 to R17, R6 to R18, R7 to R19, R1 to R2, R16 to R20, R17 to R21, R2 to R3, R3 to R4, R18 to R5, R19 to R6, R20 to R7, R21 to R8, R8 to R9
Connections:
- net PERSONAL_ALERT_BUTTON_LEFT: now also S1.1
- net PERSONAL_ALERT_BUTTON_RIGHT: now also S3.1
- net VBUS_READ: now also U1.8 (D7); no longer U1.3 (D2)
- net at JP4.1 (A): now also S2.1
- net at C1.1, C10.1, C11.1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: now also IC1.2 (VDD), IC10.2 (VDD), IC2.2 (VDD), IC3.2 (VDD), IC4.2 (VDD), IC5.2 (VDD), IC6.2 (VDD), IC7.2 (VDD), IC8.2 (VDD), IC9.2 (VDD)
- net at R1.2: now also IC1.1 (DIN)
- net at JP25.2 (B), TP15.1: now also LS1.1 (+)
- net at J1.2 (Pin_2): now also U1.3 (D2); no longer U1.8 (D7)
- net USB_DN: now reaches J3.A7 (DN1), J3.B7 (DN2), U1.21 (USB_DN)
- net USB_DP: now reaches J3.A6 (DP1), J3.B6 (DP2), U1.22 (USB_DP)
- net at JP26.2 (B), TP16.1: now also LS1.2 (-)
- net at R21.2: now also LED2.1 (K)
- net at JP24.2 (B): now also LED2.2 (A)
- net at R4.2: now also LED1.1 (K)
- net at JP3.2 (B): now also LED1.2 (A)
- net -BATT renamed GND
- net GND: now also IC1.4 (GND), IC10.4 (GND), IC2.4 (GND), IC3.4 (GND), IC4.4 (GND), IC5.4 (GND), IC6.4 (GND), IC7.4 (GND), IC8.4 (GND), IC9.4 (GND), S1.2, S1.3 (GND), S1.4 (GND__1), S2.2, S2.3 (GND), S2.4 (GND__1), S3.2, S3.3 (GND), S3.4 (GND__1)
- new net: IC7.3 (DOUT), IC8.1 (DIN)
- new net: IC8.3 (DOUT), IC9.1 (DIN)
- new net: IC6.3 (DOUT), IC7.1 (DIN)
- new net: IC2.3 (DOUT), IC3.1 (DIN)
- new net: IC3.3 (DOUT), IC4.1 (DIN)
- new net: IC4.3 (DOUT), IC5.1 (DIN)
- new net: IC10.1 (DIN), IC9.3 (DOUT)
- new net: IC5.3 (DOUT), IC6.1 (DIN)
- new net: IC1.3 (DOUT), IC2.1 (DIN)
Other:
- note added: "ATECC608A can be isolated and driven via test pads by cutting JP6,10,11,17,20"
- note added: "BATTERY CHARGING INFERENCE (VBUS HIGH IF POWERED OVER USB)"
- note added: "Buzzer can be isolated and driven via test pads by cutting JP15,22,25,26"
- note added: "CRYPTO"
- note added: "DRV2605L can be isolated and driven via test pads by cutting JP7,12,13,14,18,21,23"
- note added: "MAX17048 can be isolated and driven via test pads by cutting JP5,8,9,16,19,24,27"
- note removed: "BATTERY CHARGING INFERENCE (VUSB HIGH IF POWERED OVER USB)"
- note removed: "Buzzer can be isolated and driven via test pads by cutting JP5 and JP6"
- note removed: "DRV2605L can be isolated and driven via test pads by cutting JP11, JP16, JP17, JP18, JP21, JP24"
- note removed: "MAX17048 can be isolated and driven via test pads by cutting JP10, JP14, JP15, JP20, JP23"
- note removed: "MAX17048 can be isolated and driven via test pads by cutting JP9, JP12, JP13,JP10, JP22"
- moved on the sheet: C1, C10, C11, C12, C13, C14, C15, C16, C17, C18, C19, C2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

Commit message: Update PCB BOM exclusions and export manufacturing artifacts.
Mark DNP/non-BOM parts on the schematic and add the exported BOM CSV plus STEP model.
Parts:
- TP1, TP10, TP11, TP12, TP13, TP14, TP15, TP16, TP2, TP3, TP4, TP5, TP6, TP7, TP8, TP9: now left out of the parts list
- U1: now not fitted
Changed lines of the file:
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@@
 		(body_style 1)
 		(exclude_from_sim no)
-		(in_bom yes)
+		(in_bom no)
 		(on_board yes)
 		(in_pos_files yes)
@@
 		(on_board yes)
 		(in_pos_files yes)
-		(dnp no)
+		(dnp yes)
 		(property "Reference" "U1"
 			(at 215.9 174.244 90)
@@
 		(body_style 1)
 		(exclude_from_sim no)
-		(in_bom yes)
+		(in_bom no)
 		(on_board yes)
 		(in_pos_files yes)
@@
 		(body_style 1)
 		(exclude_from_sim no)
-		(in_bom yes)
+		(in_bom no)
 		(on_board yes)
 		(in_pos_files yes)
@@
 		(body_style 1)
 		(exclude_from_sim no)
-		(in_bom yes)
+		(in_bom no)
 		(on_board yes)
 		(in_pos_files yes)
@@
 		(body_style 1)
 		(exclude_from_sim no)
-		(in_bom yes)
+		(in_bom no)
 		(on_board yes)
 		(in_pos_files yes)
@@
 		(body_style 1)
 		(exclude_from_sim no)
-		(in_bom yes)
+		(in_bom no)
 		(on_board yes)
 		(in_pos_files yes)
@@
 		(body_style 1)
 		(exclude_from_sim no)
-		(in_bom yes)
+		(in_bom no)
 		(on_board yes)
 		(in_pos_files yes)
@@
 		(body_style 1)
 		(exclude_from_sim no)
-		(in_bom yes)
+		(in_bom no)
 		(on_board yes)
 		(in_pos_files yes)
@@
 			)
 		)
-		(property "Manufacturer" ""
+		(property "MANUFACTURER" ""
 			(at 76.2 207.01 90)
 			(hide yes)
@@
 		(body_style 1)
 		(exclude_from_sim no)
-		(in_bom yes)
+		(in_bom no)
 		(on_board yes)
 		(in_pos_files yes)
@@
 		(body_style 1)
 		(exclude_from_sim no)
-		(in_bom yes)
+		(in_bom no)
 		(on_board yes)
 		(in_pos_files yes)
@@
 		(body_style 1)
 		(exclude_from_sim no)
-		(in_bom yes)
+		(in_bom no)
 		(on_board yes)
 		(in_pos_files yes)
@@
 		(body_style 1)
 		(exclude_from_sim no)
-		(in_bom yes)
+		(in_bom no)
 		(on_board yes)
 		(in_pos_files yes)
@@
 		(body_style 1)
 		(exclude_from_sim no)
-		(in_bom yes)
+		(in_bom no)
 		(on_board yes)
 		(in_pos_files yes)
@@
 		(body_style 1)
 		(exclude_from_sim no)
-		(in_bom yes)
+		(in_bom no)
 		(on_board yes)
 		(in_pos_files yes)
@@
 			)
 		)
-		(property "Manufacturer" ""
+		(property "MANUFACTURER" ""
 			(at 530.86 121.92 90)
 			(hide yes)
@@
 		(body_style 1)
 		(exclude_from_sim no)
-		(in_bom yes)
+		(in_bom no)
 		(on_board yes)
 		(in_pos_files yes)
@@
 		(body_style 1)
 		(exclude_from_sim no)
-		(in_bom yes)
+		(in_bom no)
 		(on_board yes)
 		(in_pos_files yes)
